File: PCB/LCRDT-Tester.kicad_pcb (KiCad board)
At the start: 2 copper layers, 30 x 50.1 mm, 19 parts, among them J1 Test, J2 Disp

Commit message: upload gerber, drill and different export files
Parts:
- renumbered REF** to REF7**, REF** to REF8**
Changed lines of the file:
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@@
       (sketchpadsonfab true)
       (subtractmaskfromsilk false)
-      (outputformat 4)
+      (outputformat 1)
       (mirror false)
       (drillshape 0)
       (scaleselection 1)
-      (outputdirectory "")
+      (outputdirectory "C:/github/LCRDT-Tester/PCB/gbr/")
     )
   )
@@
         (effects (font (size 1 1) (thickness 0.15)))
     )
-    (fp_text user "${REFERENCE}" (at 0 2.54 90) (layer "F.Fab")
+    (fp_text user "${REFERENCE}" (at -2.2795 -0.71 180) (layer "F.Fab")
         (effects (font (size 1 1) (thickness 0.15)))
     )
@@
         (effects (font (size 0.75 0.75) (thickness 0.15)) (justify mirror))
     )
-    (fp_text user "${REFERENCE}" (at -2.49 0.26 90) (layer "B.Fab")
-        (effects (font (size 0.72 0.72) (thickness 0.108)) (justify mirror))
-    )
-    (fp_text user "${REFERENCE}" (at -2.49 0.2 90) (layer "F.Fab")
-        (effects (font (size 0.72 0.72) (thickness 0.108)))
+    (fp_text user "${REFERENCE}" (at -2.466 0.07 90) (layer "F.Fab")
+        (effects (font (size 0.75 0.75) (thickness 0.125) bold))
     )
     (fp_line (start 0.94 0) (end 1.89 0)
@@
         (effects (font (size 0.5 0.5) (thickness 0.125)))
     )
-    (fp_text user "${REFERENCE}" (at 6.096 2.5095) (layer "F.Fab")
+    (fp_text user "${REFERENCE}" (at 5.96 2.748) (layer "F.Fab")
         (effects (font (size 1 1) (thickness 0.15)))
     )
@@
     )
     (fp_text user "${REFERENCE}" (at -2.49 0.07 90) (layer "F.Fab")
-        (effects (font (size 0.72 0.72) (thickness 0.108)))
+        (effects (font (size 0.75 0.75) (thickness 0.125) bold))
     )
     (fp_line (start 0.94 0) (end 1.89 0)
@@
         (effects (font (size 0.75 0.75) (thickness 0.15) bold) (justify mirror))
     )
-    (fp_text user "${REFERENCE}" (at 1.524 -1.8035 90) (layer "F.Fab")
-        (effects (font (size 0.5 0.5) (thickness 0.108)))
+    (fp_text user "${REFERENCE}" (at -2.442 -0.14 90) (layer "F.Fab")
+        (effects (font (size 0.75 0.75) (thickness 0.125) bold))
     )
     (fp_line (start 0.94 0) (end 1.89 0)
@@
     (property "ki_keywords" "switch normally-open pushbutton push-button")
     (attr through_hole)
-    (fp_text reference "Start" (at 8.96 1.33) (layer "F.SilkS")
+    (fp_text reference "Start" (at 8.86 2.4) (layer "F.SilkS")
         (effects (font (size 0.75 0.75) (thickness 0.15)))
     )
@@
         (effects (font (size 0.75 0.75) (thickness 0.15)))
     )
-    (fp_text user "${REFERENCE}" (at 0 3.81 90) (layer "F.Fab")
+    (fp_text user "${REFERENCE}" (at -2.409 -0.14 180) (layer "F.Fab")
         (effects (font (size 1 1) (thickness 0.15)))
     )
@@
     (tags "mounting hole 3.2mm m3 din965")
     (attr exclude_from_pos_files exclude_from_bom)
-    (fp_text reference "REF9**" (at 0 -3.8) (layer "F.Fab")
+    (fp_text reference "REF9**" (at -7.44 3.53) (layer "F.Fab") hide
         (effects (font (size 1 1) (thickness 0.15)))
     )
-    (fp_text value "MountingHole_3.2mm_M3_DIN965_Pad" (at 0 3.8) (layer "F.Fab")
+    (fp_text value "MountingHole_3.2mm_M3_DIN965_Pad" (at -4.89 5.67 90) (layer "F.Fab") hide
         (effects (font (size 1 1) (thickness 0.15)))
     )
-    (fp_text user "${REFERENCE}" (at 0 0) (layer "F.Fab")
+    (fp_text user "${REFERENCE}" (at -0.17 -4.18) (layer "F.Fab")
         (effects (font (size 1 1) (thickness 0.15)))
     )
@@
         (effects (font (size 0.75 0.75) (thickness 0.15) bold))
     )
-    (fp_text value "SW_Push" (at 4.4 3.7) (layer "F.Fab")
+    (fp_text value "SW_Push" (at -4.69 1.43) (layer "F.Fab")
         (effects (font (size 1 1) (thickness 0.15)))
     )
-    (fp_text user "${REFERENCE}" (at 3 0) (layer "F.Fab")
+    (fp_text user "${REFERENCE}" (at 3.25 1.75) (layer "F.Fab")
         (effects (font (size 1 1) (thickness 0.15)))
     )
@@
     (tags "Logo WEEE")
     (attr exclude_from_pos_files exclude_from_bom)
-    (fp_text reference "REF**" (at 0 0) (layer "B.SilkS") hide
+    (fp_text reference "REF7**" (at 0 0) (layer "B.SilkS") hide
         (effects (font (size 1 1) (thickness 0.15)) (justify mirror))
     )
@@
     (tags "Logo KiCad")
     (attr exclude_from_pos_files exclude_from_bom)
-    (fp_text reference "REF**" (at 0 5.08 90) (layer "B.SilkS") hide
+    (fp_text reference "REF8**" (at 0 5.08 90) (layer "B.SilkS") hide
         (effects (font (size 1 1) (thickness 0.15)) (justify mirror))
     )
@@
     (effects (font (size 0.5 0.5) (thickness 0.125)) (justify mirror))
   )
-  (gr_text "Start" (at 97.26 137.09) (layer "B.SilkS")
+  (gr_text "Start" (at 96.18 137.02) (layer "B.SilkS")
     (effects (font (size 0.75 0.75) (thickness 0.15)) (justify mirror))
   )
