File: PCB/LCRDT-Tester.kicad_pcb (KiCad board)
At the start: 2 copper layers, 30 x 50.1 mm, 19 parts, among them J1 Test, J2 Disp

Commit message: cleanups+Mountingholes
Parts:
- A1: footprint Module:Arduino_Nano -> Module:Arduino_Nano_WithMountingHoles
- moved G21 0.96 mm to (111.5, 126.3)
- moved Reset 0.09 mm to (108.1, 90.8)
- moved A1 0.08 mm to (118.4, 132.3)
- moved R6 0.07 mm to (107.7, 94.6)
Routing:
- net Net-(A1-~{RESET}-Pad28): track 65.1 -> 62.5 mm
- net Net-(A1-A0): track 29.1 -> 29.8 mm
Other:
- board text added: "LCRDT-Tester"
- board text added: "Rev. 0.31 © 04/2023"
- board text added: "Rev. 0.31 © 04/2024"
- board text added: "WodoWiesel"
- board text removed: "O"
- board text removed: "Rev. 0.3 © 10/2023"
